File: mote-hardware/motor.kicad_sch (KiCad schematic)
At the start: 10 parts, among them J7 left_motor, J8 right_motor, U3 DRV8833PWP

Commit message: Finish routing
Parts:
- removed U3: DRV8833PWP, Package_SO:HTSSOP-16-1EP_4.4x5mm_P0.65mm_EP3.4x5mm_Mask2.46x2.31mm_ThermalVias, symbol Driver_Motor:DRV8833PWP
- added U5: DRV8833PW, Package_SO:TSSOP-16-1EP_4.4x5mm_P0.65mm, symbol Driver_Motor:DRV8833PW
Connections:
- net GND: now also U5.13 (GND)
- net V_MOTOR: now also U5.12 (VM)
- net left_motor_a: now also U5.16 (AIN1)
- net left_motor_b: now also U5.15 (AIN2)
- net right_motor_a: now also U5.9 (BIN1)
- net right_motor_b: now also U5.10 (BIN2)
- net sleep: now also U5.1 (~{SLEEP})
- net at J8.5 (Pin_5): now also U5.7 (BOUT1)
- net at J8.6 (Pin_6): now also U5.5 (BOUT2)
- net at J7.5 (Pin_5): now also U5.2 (AOUT1)
- net at J7.6 (Pin_6): now also U5.4 (AOUT2)
- net at R12.2: now also U5.6 (BISEN)
- net at C19.1: now also U5.11 (VCP)
- net at C20.2: now also U5.14 (VINT)
- net at R11.2: now also U5.3 (AISEN)
Changed lines of the file:
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@@
 	)
 	(symbol
-		(lib_id "Driver_Motor:DRV8833PWP")
+		(lib_id "Driver_Motor:DRV8833PW")
 		(at 152.4 106.68 0)
 		(unit 1)
@@
 		(dnp no)
 		(fields_autoplaced yes)
-		(property "Reference" "U3"
+		(property "Reference" "U5"
 			(at 154.5433 121.92 0)
 			(effects
@@
 			)
 		)
-		(property "Value" "DRV8833PWP"
+		(property "Value" "DRV8833PW"
 			(at 154.5433 124.46 0)
 			(effects
@@
 			)
 		)
-		(property "Footprint" "Package_SO:HTSSOP-16-1EP_4.4x5mm_P0.65mm_EP3.4x5mm_Mask2.46x2.31mm_ThermalVias"
-			(at 157.48 121.92 0)
+		(property "Footprint" "Package_SO:TSSOP-16-1EP_4.4x5mm_P0.65mm"
+			(at 157.48 124.46 0)
 			(effects
 				(font
@@
 		)
 		(property "Datasheet" "http://www.ti.com/lit/ds/symlink/drv8833.pdf"
-			(at 157.48 124.46 0)
+			(at 157.48 127 0)
 			(effects
 				(font
@@
 			)
 		)
-		(property "Description" "Dual H-Bridge Motor Driver, HTSSOP-16"
+		(property "Description" "Dual H-Bridge Motor Driver, TSSOP-16"
 			(at 152.4 106.68 0)
 			(effects
@@
 			)
 		)
+		(pin "10"
+		)
 		(pin "13"
+		)
+		(pin "12"
+		)
+		(pin "8"
+		)
+		(pin "4"
+		)
+		(pin "2"
+		)
+		(pin "14"
+		)
+		(pin "7"
+		)
+		(pin "6"
+		)
+		(pin "5"
 		)
 		(pin "11"
@@
 		(pin "1"
 		)
-		(pin "3"
-		)
-		(pin "14"
+		(pin "15"
 		)
 		(pin "9"
 		)
-		(pin "2"
+		(pin "16"
 		)
-		(pin "17"
-		)
-		(pin "10"
-		)
-		(pin "15"
-		)
-		(pin "7"
-		)
-		(pin "8"
-		)
-		(pin "12"
-		)
-		(pin "5"
-		)
-		(pin "4"
-		)
-		(pin "6"
-		)
-		(pin "16"
+		(pin "3"
 		)
 		(instances
 			(project ""
 				(path "/94683f5c-9cd9-448e-be96-9792537b5cb8/332292ea-bd81-44ca-9f8d-1cb79fb18ef4"
-					(reference "U3")
+					(reference "U5")
 					(unit 1)
 				)

Commit message: Finish selecting LCSC components
Parts:
- C19, C20, C22: footprint Capacitor_SMD:C_0402_1005Metric -> PCM_JLCPCB:C_0402
- C2: footprint Capacitor_SMD:C_1206_3216Metric -> PCM_JLCPCB:C_1206
- C21: footprint Capacitor_SMD:C_0805_2012Metric -> PCM_JLCPCB:C_0805
- R11, R12: footprint Resistor_SMD:R_0402_1005Metric -> PCM_JLCPCB:R_0402
Changed lines of the file:
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@@
 			)
 		)
-		(property "Footprint" "Capacitor_SMD:C_1206_3216Metric"
+		(property "Footprint" "PCM_JLCPCB:C_1206"
 			(at 167.3352 71.12 0)
 			(effects
@@
 		)
 		(instances
-			(project ""
+			(project "mote-hardware"
 				(path "/94683f5c-9cd9-448e-be96-9792537b5cb8/332292ea-bd81-44ca-9f8d-1cb79fb18ef4"
 					(reference "C2")
@@
 			)
 		)
-		(property "Footprint" "Capacitor_SMD:C_0805_2012Metric"
+		(property "Footprint" "PCM_JLCPCB:C_0805"
 			(at 179.3748 63.5 0)
 			(effects
@@
 			)
 		)
-		(property "Footprint" "Capacitor_SMD:C_0402_1005Metric"
+		(property "Footprint" "PCM_JLCPCB:C_0402"
 			(at 192.0748 63.5 0)
 			(effects
@@
 		)
 		(instances
-			(project ""
+			(project "mote-hardware"
 				(path "/94683f5c-9cd9-448e-be96-9792537b5cb8/332292ea-bd81-44ca-9f8d-1cb79fb18ef4"
 					(reference "J7")
@@
 			)
 		)
-		(property "Footprint" "Resistor_SMD:R_0402_1005Metric"
+		(property "Footprint" "PCM_JLCPCB:R_0402"
 			(at 127 105.918 90)
 			(effects
@@
 		)
 		(instances
-			(project ""
+			(project "mote-hardware"
 				(path "/94683f5c-9cd9-448e-be96-9792537b5cb8/332292ea-bd81-44ca-9f8d-1cb79fb18ef4"
 					(reference "U5")
@@
 			)
 		)
-		(property "Footprint" "Capacitor_SMD:C_0402_1005Metric"
+		(property "Footprint" "PCM_JLCPCB:C_0402"
 			(at 137.4648 77.47 0)
 			(effects
@@
 			)
 		)
-		(property "Footprint" "Resistor_SMD:R_0402_1005Metric"
+		(property "Footprint" "PCM_JLCPCB:R_0402"
 			(at 127 103.378 90)
 			(effects
@@
 		)
 		(instances
-			(project ""
+			(project "mote-hardware"
 				(path "/94683f5c-9cd9-448e-be96-9792537b5cb8/332292ea-bd81-44ca-9f8d-1cb79fb18ef4"
 					(reference "R11")
@@
 			)
 		)
-		(property "Footprint" "Capacitor_SMD:C_0402_1005Metric"
+		(property "Footprint" "PCM_JLCPCB:C_0402"
 			(at 167.9448 85.09 0)
 			(effects

Commit message: Update date and github link
Other:
- company: github.com/usedhondacivic/mote -> github.com/empriselab/mote-core
Changed lines of the file:
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@@
 	(title_block
 		(title "Mote")
-		(date "2026-03-22")
+		(date "2026-03-31")
 		(rev "V0.0.0")
-		(company "github.com/usedhondacivic/mote")
+		(company "github.com/empriselab/mote-core")
 	)
 	(text "1A current limit\n[CHOP = (0.2V / RSENSE)]"
