File: mote-hardware/status_indicator.kicad_sch (KiCad schematic)
At the start: 4 parts

Commit message: Get pcb ready for first prototype order (#31)
Co-authored-by: Kyle Mui <44453997+KyleMui@users.noreply.github.com>
Parts:
- added D1, D2: LED, LED_SMD:LED_0603_1608Metric, symbol Device:LED
- added R16, R17: 2.2k, PCM_JLCPCB:R_0402, symbol Device:R
- R13: footprint Resistor_SMD:R_0603_1608Metric_Pad0.98x0.95mm_HandSolder -> PCM_JLCPCB:R_0603
Connections:
- net +5v: now also D1.2 (A)
- net GND: now also R16.2, R17.2
- new net: D1.1 (K), R16.1
- new net: D2.1 (K), R17.1
- new net +3v3: D2.2 (A)
Other:
- note added: "Power indication"
- company: github.com/usedhondacivic/mote -> github.com/empriselab/mote-core
- moved on the sheet: D3, D4, D5, R13

Commit message: Assign LCSC part numbers
Parts:
- D1, D2: LCSC (none) -> C2290
- R13: LCSC (none) -> C23204
- R16, R17: LCSC (none) -> C25879
Changed lines of the file:
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@@
 			)
 		)
-		(property "LCSC" ""
+		(property "LCSC" "C23204"
 			(at 72.39 104.14 0)
 			(effects
@@
 			)
 		)
+		(property "LCSC" "C2290"
+			(at 204.47 97.79 90)
+			(effects
+				(font
+					(size 1.27 1.27)
+				)
+				(hide yes)
+			)
+		)
 		(pin "2"
 		)
@@
 			)
 		)
+		(property "LCSC" "C25879"
+			(at 215.9 109.22 0)
+			(effects
+				(font
+					(size 1.27 1.27)
+				)
+				(hide yes)
+			)
+		)
 		(pin "2"
 		)
@@
 			)
 		)
+		(property "LCSC" "C25879"
+			(at 204.47 109.22 0)
+			(effects
+				(font
+					(size 1.27 1.27)
+				)
+				(hide yes)
+			)
+		)
 		(pin "2"
 		)
@@
 			(effects
 				(font
+					(size 1.27 1.27)
+				)
+				(hide yes)
+			)
+		)
+		(property "LCSC" "C2290"
+			(at 215.9 97.79 90)
+			(effects
+				(font
