File: mote-hardware/status_indicator.kicad_sch (KiCad schematic)
At the start: 0 parts

Commit message: Implement motor, power, imu, status LED schematics
Parts:
- added D3, D4, D5: WS2812B-2020, LED_SMD:LED_WS2812B-2020_PLCC4_2.0x2.0mm, symbol LED:WS2812B-2020
- added R13: 560, Resistor_SMD:R_0603_1608Metric_Pad0.98x0.95mm_HandSolder, symbol Device:R
Connections:
- new net: D3.3 (DIN), R13.2
- new net: D4.1 (DOUT), D5.3 (DIN)
- new net: D3.1 (DOUT), D4.3 (DIN)
- new net +5v: D3.4 (VDD), D4.4 (VDD), D5.4 (VDD)
- new net GND: D3.2 (VSS), D4.2 (VSS), D5.2 (VSS)
- new net rx: R13.1
- no-connect marks 0 -> 1
Other:
- note added: "Neopixels"

Commit message: First draft schematic complete
Other:
- company: (none) -> github.com/usedhondacivic/mote
- title: (none) -> Mote
Changed lines of the file:
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@@
 	(generator_version "9.0")
 	(paper "A4")
+	(title_block
+		(title "Mote")
+		(date "2025-12-30")
+		(rev "V0.0.0")
+		(company "github.com/usedhondacivic/mote")
+	)
 	(text "Neopixels"
 		(exclude_from_sim no)

Commit message: added led and did checks
Parts:
- added D1, D2: LED, LED_SMD:LED_0603_1608Metric, symbol Device:LED
- added R16, R17: 2.2k, Resistor_SMD:R_0402_1005Metric, symbol Device:R
Connections:
- net +5v: now also D1.2 (A)
- net GND: now also R16.2, R17.2
- new net: D1.1 (K), R16.1
- new net: D2.1 (K), R17.1
- new net +3v3: D2.2 (A)

Commit message: Finish selecting LCSC components
Parts:
- R13: footprint Resistor_SMD:R_0603_1608Metric_Pad0.98x0.95mm_HandSolder -> PCM_JLCPCB:R_0603
- R16, R17: footprint Resistor_SMD:R_0402_1005Metric -> PCM_JLCPCB:R_0402
Other:
- note added: "Power indication"
- moved on the sheet: D3, D4, D5, R13

Commit message: Update date and github link
Other:
- company: github.com/usedhondacivic/mote -> github.com/empriselab/mote-core
Changed lines of the file:
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@@
 	(title_block
 		(title "Mote")
-		(date "2026-03-22")
+		(date "2026-03-31")
 		(rev "V0.0.0")
-		(company "github.com/usedhondacivic/mote")
+		(company "github.com/empriselab/mote-core")
 	)
 	(text "Neopixels"

Commit message: Hardware v0.0.0 order (#36)
Parts:
- D1, D2: LCSC (none) -> C2290
- R13: LCSC (none) -> C23204
- R16, R17: LCSC (none) -> C25879
Changed lines of the file:
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@@
 			)
 		)
-		(property "LCSC" ""
+		(property "LCSC" "C23204"
 			(at 72.39 104.14 0)
+			(effects
+				(font
+					(size 1.27 1.27)
+				)
+				(hide yes)
+			)
+		)
+		(property "JLCPCB_CORRECTION" ""
+			(at 72.39 104.14 90)
 			(effects
 				(font
@@
 			)
 		)
+		(property "LCSC" "C2290"
+			(at 204.47 97.79 90)
+			(effects
+				(font
+					(size 1.27 1.27)
+				)
+				(hide yes)
+			)
+		)
+		(property "JLCPCB_CORRECTION" ""
+			(at 204.47 97.79 90)
+			(effects
+				(font
+					(size 1.27 1.27)
+				)
+				(hide yes)
+			)
+		)
 		(pin "2"
 		)
@@
 			)
 		)
+		(property "JLCPCB_CORRECTION" ""
+			(at 134.62 104.14 0)
+			(effects
+				(font
+					(size 1.27 1.27)
+				)
+				(hide yes)
+			)
+		)
 		(pin "1"
 		)
@@
 			)
 		)
+		(property "JLCPCB_CORRECTION" ""
+			(at 87.63 104.14 0)
+			(effects
+				(font
+					(size 1.27 1.27)
+				)
+				(hide yes)
+			)
+		)
 		(pin "1"
 		)
@@
 		)
 		(property "LCSC" "C965555"
+			(at 111.76 104.14 0)
+			(effects
+				(font
+					(size 1.27 1.27)
+				)
+				(hide yes)
+			)
+		)
+		(property "JLCPCB_CORRECTION" ""
 			(at 111.76 104.14 0)
 			(effects
@@
 			)
 		)
+		(property "LCSC" "C25879"
+			(at 215.9 109.22 0)
+			(effects
+				(font
+					(size 1.27 1.27)
+				)
+				(hide yes)
+			)
+		)
+		(property "JLCPCB_CORRECTION" ""
+			(at 215.9 109.22 0)
+			(effects
+				(font
+					(size 1.27 1.27)
+				)
+				(hide yes)
+			)
+		)
 		(pin "2"
 		)
@@
 			)
 		)
+		(property "LCSC" "C25879"
+			(at 204.47 109.22 0)
+			(effects
+				(font
+					(size 1.27 1.27)
+				)
+				(hide yes)
+			)
+		)
+		(property "JLCPCB_CORRECTION" ""
+			(at 204.47 109.22 0)
+			(effects
+				(font
+					(size 1.27 1.27)
+				)
+				(hide yes)
+			)
+		)
 		(pin "2"
 		)
@@
 			(effects
 				(font
+					(size 1.27 1.27)
+				)
+				(hide yes)
+			)
+		)
+		(property "LCSC" "C2290"
+			(at 215.9 97.79 90)
+			(effects
+				(font
+					(size 1.27 1.27)
+				)
+				(hide yes)
+			)
+		)
+		(property "JLCPCB_CORRECTION" ""
+			(at 215.9 97.79 90)
+			(effects
+				(font
