File: mote-hardware/rp_lidar_c1.kicad_sch (KiCad schematic)
At the start: 5 parts, among them J2 JST_XH2.54-SP

Commit message: Get pcb ready for first prototype order
Parts:
- J2: footprint Connector_JST:JST_XH_S5B-XH-A_1x05_P2.50mm_Horizontal -> Connector_JST:JST_XH_B5B-XH-A_1x05_P2.50mm_Vertical
Changed lines of the file:
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@@
 	(title_block
 		(title "Mote")
-		(date "2025-12-30")
+		(date "2026-03-22")
 		(rev "V0.0.0")
 		(company "github.com/usedhondacivic/mote")
@@
 			)
 		)
-		(property "Footprint" "Connector_JST:JST_XH_S5B-XH-A_1x05_P2.50mm_Horizontal"
+		(property "Footprint" "Connector_JST:JST_XH_B5B-XH-A_1x05_P2.50mm_Vertical"
 			(at 110.49 100.33 0)
 			(effects

Commit message: Update date and github link
Other:
- company: github.com/usedhondacivic/mote -> github.com/empriselab/mote-core
Changed lines of the file:
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@@
 	(title_block
 		(title "Mote")
-		(date "2026-03-22")
+		(date "2026-03-31")
 		(rev "V0.0.0")
-		(company "github.com/usedhondacivic/mote")
+		(company "github.com/empriselab/mote-core")
 	)
 	(text "UART"

Commit message: Hardware v0.0.0 order (#36)
Parts:
- H1, H2, H3, H4: now not fitted
- J2: LCSC (none) -> C157991
Changed lines of the file:
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@@
 		(in_bom no)
 		(on_board yes)
-		(dnp no)
+		(dnp yes)
 		(fields_autoplaced yes)
 		(property "Reference" "H1"
@@
 		)
 		(property "Description" "Mounting Hole without connection"
+			(at 165.1 91.44 0)
+			(effects
+				(font
+					(size 1.27 1.27)
+				)
+				(hide yes)
+			)
+		)
+		(property "JLCPCB_CORRECTION" ""
 			(at 165.1 91.44 0)
 			(effects
@@
 		(in_bom no)
 		(on_board yes)
-		(dnp no)
+		(dnp yes)
 		(fields_autoplaced yes)
 		(property "Reference" "H3"
@@
 		)
 		(property "Description" "Mounting Hole without connection"
+			(at 165.1 101.6 0)
+			(effects
+				(font
+					(size 1.27 1.27)
+				)
+				(hide yes)
+			)
+		)
+		(property "JLCPCB_CORRECTION" ""
 			(at 165.1 101.6 0)
 			(effects
@@
 			)
 		)
+		(property "LCSC" "C157991"
+			(at 110.49 100.33 0)
+			(effects
+				(font
+					(size 1.27 1.27)
+				)
+				(hide yes)
+			)
+		)
+		(property "JLCPCB_CORRECTION" ""
+			(at 110.49 100.33 0)
+			(effects
+				(font
+					(size 1.27 1.27)
+				)
+				(hide yes)
+			)
+		)
 		(pin "2"
 		)
@@
 		(in_bom no)
 		(on_board yes)
-		(dnp no)
+		(dnp yes)
 		(fields_autoplaced yes)
 		(property "Reference" "H2"
@@
 		)
 		(property "Description" "Mounting Hole without connection"
+			(at 165.1 96.52 0)
+			(effects
+				(font
+					(size 1.27 1.27)
+				)
+				(hide yes)
+			)
+		)
+		(property "JLCPCB_CORRECTION" ""
 			(at 165.1 96.52 0)
 			(effects
@@
 		(in_bom no)
 		(on_board yes)
-		(dnp no)
+		(dnp yes)
 		(fields_autoplaced yes)
 		(property "Reference" "H4"
@@
 			(at 165.1 106.68 0)
 			(effects
+				(font
+					(size 1.27 1.27)
+				)
+				(hide yes)
+			)
+		)
+		(property "JLCPCB_CORRECTION" ""
+			(at 165.1 106.68 0)
+			(effects
