File: mote-hardware/rp_lidar_c1.kicad_sch (KiCad schematic)
At the start: 0 parts

Commit message: Implement motor, power, imu, status LED schematics
Parts:
- added H1, H2, H3, H4: M2.5 loose, symbol Mechanical:MountingHole
- added J2: JST_XH2.54-SP, symbol Connector_Generic:Conn_01x05
Connections:
- new net +5v: J2.1 (Pin_1)
- new net GND: J2.4 (Pin_4)
- new net RX: J2.3 (Pin_3)
- new net TX: J2.2 (Pin_2)
- no-connect marks 0 -> 1
Other:
- note added: "Mounting"
- note added: "UART"

Commit message: First draft schematic complete
Other:
- company: (none) -> github.com/usedhondacivic/mote
- title: (none) -> Mote
Changed lines of the file:
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@@
 	(generator_version "9.0")
 	(paper "A4")
+	(title_block
+		(title "Mote")
+		(date "2025-12-30")
+		(rev "V0.0.0")
+		(company "github.com/usedhondacivic/mote")
+	)
 	(text "UART"
 		(exclude_from_sim no)

Commit message: Footprint assignments
Parts:
- H1, H2, H3, H4: footprint (none) -> MountingHole:MountingHole_2.7mm_M2.5
- J2: footprint (none) -> Connector_JST:JST_XH_S5B-XH-A_1x05_P2.50mm_Horizontal
Changed lines of the file:
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@@
 			)
 		)
-		(property "Footprint" ""
+		(property "Footprint" "MountingHole:MountingHole_2.7mm_M2.5"
 			(at 165.1 91.44 0)
 			(effects
@@
 			)
 		)
-		(property "Footprint" ""
+		(property "Footprint" "MountingHole:MountingHole_2.7mm_M2.5"
 			(at 165.1 101.6 0)
 			(effects
@@
 			)
 		)
-		(property "Footprint" ""
+		(property "Footprint" "Connector_JST:JST_XH_S5B-XH-A_1x05_P2.50mm_Horizontal"
 			(at 110.49 100.33 0)
 			(effects
@@
 			)
 		)
-		(property "Footprint" ""
+		(property "Footprint" "MountingHole:MountingHole_2.7mm_M2.5"
 			(at 165.1 96.52 0)
 			(effects
@@
 			)
 		)
-		(property "Footprint" ""
+		(property "Footprint" "MountingHole:MountingHole_2.7mm_M2.5"
 			(at 165.1 106.68 0)
 			(effects

Commit message: Get pcb ready for first prototype order (#31)
Co-authored-by: Kyle Mui <44453997+KyleMui@users.noreply.github.com>
Parts:
- J2: footprint Connector_JST:JST_XH_S5B-XH-A_1x05_P2.50mm_Horizontal -> Connector_JST:JST_XH_B5B-XH-A_1x05_P2.50mm_Vertical
Other:
- company: github.com/usedhondacivic/mote -> github.com/empriselab/mote-core
Changed lines of the file:
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@@
 	(title_block
 		(title "Mote")
-		(date "2025-12-30")
+		(date "2026-03-31")
 		(rev "V0.0.0")
-		(company "github.com/usedhondacivic/mote")
+		(company "github.com/empriselab/mote-core")
 	)
 	(text "UART"
@@
 		)
 		(instances
-			(project ""
+			(project "mote-hardware"
 				(path "/94683f5c-9cd9-448e-be96-9792537b5cb8/0a44614a-b30e-47eb-9b35-85ffdcfad2e9"
 					(reference "H1")
@@
 			)
 		)
-		(property "Footprint" "Connector_JST:JST_XH_S5B-XH-A_1x05_P2.50mm_Horizontal"
+		(property "Footprint" "Connector_JST:JST_XH_B5B-XH-A_1x05_P2.50mm_Vertical"
 			(at 110.49 100.33 0)
 			(effects
@@
 		)
 		(instances
-			(project ""
+			(project "mote-hardware"
 				(path "/94683f5c-9cd9-448e-be96-9792537b5cb8/0a44614a-b30e-47eb-9b35-85ffdcfad2e9"
 					(reference "J2")

Commit message: Assign LCSC part numbers
Parts:
- H1, H2, H3, H4: now not fitted
- J2: LCSC (none) -> C144397
Changed lines of the file:
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@@
 		(in_bom no)
 		(on_board yes)
-		(dnp no)
+		(dnp yes)
 		(fields_autoplaced yes)
 		(property "Reference" "H1"
@@
 		(in_bom no)
 		(on_board yes)
-		(dnp no)
+		(dnp yes)
 		(fields_autoplaced yes)
 		(property "Reference" "H3"
@@
 			)
 		)
+		(property "LCSC" "C144397"
+			(at 110.49 100.33 0)
+			(effects
+				(font
+					(size 1.27 1.27)
+				)
+				(hide yes)
+			)
+		)
 		(pin "2"
 		)
@@
 		(in_bom no)
 		(on_board yes)
-		(dnp no)
+		(dnp yes)
 		(fields_autoplaced yes)
 		(property "Reference" "H2"
@@
 		(in_bom no)
 		(on_board yes)
-		(dnp no)
+		(dnp yes)
 		(fields_autoplaced yes)
 		(property "Reference" "H4"

Commit message: Fix ups
Parts:
- J2: LCSC C144397 -> C157991
Changed lines of the file:
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@@
+			)
+		)
+		(property "JLCPCB_CORRECTION" ""
+			(at 165.1 91.44 0)
+			(effects
+				(font
+					(size 1.27 1.27)
+				)
+				(hide yes)
 			)
 		)
@@
 			)
 		)
+		(property "JLCPCB_CORRECTION" ""
+			(at 165.1 101.6 0)
+			(effects
+				(font
+					(size 1.27 1.27)
+				)
+				(hide yes)
+			)
+		)
 		(instances
 			(project "mote-hardware"
@@
 			)
 		)
-		(property "LCSC" "C144397"
+		(property "LCSC" "C157991"
+			(at 110.49 100.33 0)
+			(effects
+				(font
+					(size 1.27 1.27)
+				)
+				(hide yes)
+			)
+		)
+		(property "JLCPCB_CORRECTION" ""
 			(at 110.49 100.33 0)
 			(effects
@@
 			)
 		)
+		(property "JLCPCB_CORRECTION" ""
+			(at 165.1 96.52 0)
+			(effects
+				(font
+					(size 1.27 1.27)
+				)
+				(hide yes)
+			)
+		)
 		(instances
 			(project "mote-hardware"
@@
 			(at 165.1 106.68 0)
 			(effects
+				(font
+					(size 1.27 1.27)
+				)
+				(hide yes)
+			)
+		)
+		(property "JLCPCB_CORRECTION" ""
+			(at 165.1 106.68 0)
+			(effects

Commit message: Add position corrections
Parts:
- J2: JLCPCB_CORRECTION (none) -> 0; 0; 0
Changed lines of the file:
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@@
 			)
 		)
-		(property "JLCPCB_CORRECTION" ""
+		(property "JLCPCB_CORRECTION" "0; 0; 0"
 			(at 110.49 100.33 0)
 			(effects
