File: mote-hardware/rp_lidar_c1.kicad_sch (KiCad schematic)
At the start: 5 parts, among them J2 JST_XH2.54-SP

Commit message: Update offsets
Parts:
- J2: JLCPCB_CORRECTION 0; 0; 0 -> 4.953; 0; 180
Changed lines of the file:
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@@
 			)
 		)
-		(property "JLCPCB_CORRECTION" "0; 0; 0"
+		(property "JLCPCB_CORRECTION" "4.953; 0; 180"
 			(at 110.49 100.33 0)
 			(effects

Commit message: Add TVS diodes
Parts:
- added D12: PTVS7V5Z1USK, Diode_SMD:Nexperia_DSN1608-2_1.6x0.8mm, symbol Diode:PTVS7V5Z1USK
- added D15, D16: PTVS5V0Z1USK, Diode_SMD:Nexperia_DSN1608-2_1.6x0.8mm, symbol Diode:PTVS5V0Z1USK
Connections:
- net +5v: now also D12.1 (K)
- net GND: now also D12.2 (A), D15.2 (A), D16.2 (A)
- net RX: now also D16.1 (K)
- net TX: now also D15.1 (K)
Other:
- note added: "ESD Protection"
- moved on the sheet: H1, H2, H3, H4, J2
